Commit message: Update urdf

File: urdf/model.urdf (robot description, URDF)
Before this commit: robot robot_name, 1 links, 0 joints
Links:
- added link camera; visual mesh filename=package://simulation/meshes/link_cam.STL
- added link left_wheel; visual mesh filename=package://simulation/meshes/link_l.STL
- added link right_wheel; visual mesh filename=package://simulation/meshes/link_r.STL
- link base_link: geometry visual mesh filename=package://simulation/meshes/base.STL
Joints:
- added joint joint_cam: type fixed, parent base_link, child camera, origin xyz=0.05 0.0 0.1 rpy=0.0 3.14159265 -1.57079632
- added joint joint_l: type continuous, parent base_link, child left_wheel, origin xyz=0.0 0.06 0.026 rpy=0.0 0.0 3.14159265, axis 0 1 0
- added joint joint_r: type continuous, parent base_link, child right_wheel, origin xyz=0.0 -0.06 0.026 rpy=0.0 0.0 0.0, axis 0 1 0

Commit message: Update mmodel.urdf

File: urdf/model.urdf (robot description, URDF)
Before this commit: robot , 4 links, 3 joints
Links:
- link base_link: mass None -> 1; geometry collision mesh filename=package://simulation/meshes/base.STL; visual mesh filename=package://simulation/meshes/base.STL
- link camera: mass None -> 0.5; geometry collision mesh filename=package://simulation/meshes/link_cam.STL; visual mesh filename=package://simulation/meshes/link_cam.STL
- link left_wheel: mass None -> 0.05; geometry collision mesh filename=package://simulation/meshes/link_l.STL; visual mesh filename=package://simulation/meshes/link_l.STL
- link right_wheel: mass None -> 0.05; geometry collision mesh filename=package://simulation/meshes/link_r.STL; visual mesh filename=package://simulation/meshes/link_r.STL

Commit message: Update Gazebo

File: urdf/model.urdf (robot description, URDF)
Before this commit: robot , 4 links, 3 joints
Joints:
- joint joint_l: origin xyz=0.0 0.06 0.026 rpy=0.0 0.0 3.14159265 -> xyz=0.0 0.06 0.026 rpy=0.0 0.0 0

File: urdf/model.xacro (robot description, xacro)
@@ -1,5 +1,4 @@
 <?xml version="1.0"?>
 <robot name="" xmlns:xacro="http://www.ros.org/wiki/xacro">
-    <!-- <xacro:property name="" value=""/> -->
     <xacro:include filename="$(find simulation)/urdf/materials.xacro" />
     <xacro:include filename="$(find simulation)/urdf/model.gazebo" />
@@ -18,7 +17,4 @@
                 <mesh filename="package://simulation/meshes/base.STL" />
             </geometry>
-            <material name="">
-                <color rgba="1.0 1.0 1.0 1.0" />
-            </material>
         </visual>
         <collision>
@@ -31,5 +27,5 @@
   <link name="left_wheel">
         <inertial>
-            <origin xyz="0.0 0.0 0.0" rpy="0 0 0" />
+            <origin xyz="0.0 0.0 0.0" rpy="0.0 0.0 0.0" />
             <mass value="0.05" />
             <inertia
@@ -39,11 +35,8 @@
         </inertial>
         <visual>
-            <origin xyz="0.0 0.0 0.0" rpy="0.0 0.0 0.0" />
+            <origin xyz="0.0 0.0 0.0" rpy="0.0 0.0 3.14159265" />
             <geometry>
                 <mesh filename="package://simulation/meshes/link_l.STL" />
             </geometry>
-            <material name="">
-                <color rgba="1.0 1.0 1.0 1.0" />
-            </material>
         </visual>
         <collision>
@@ -55,10 +48,8 @@
   </link>
     <joint name="joint_l" type="continuous">
-        <origin xyz="0.0 0.06 0.026" rpy="0.0 0.0 3.14159265" />
+        <origin xyz="0.0 0.06 0.026" rpy="0.0 0.0 0.0" />
         <parent link="base_link" />
         <child link="left_wheel" />
         <axis xyz="0 1 0" />
-        <limit effort="10000" velocity="1000"/>
-        <joint_properties damping="1.0" friction="1.0"/>
     </joint>
     <link name="right_wheel">
@@ -76,7 +67,4 @@
                 <mesh filename="package://simulation/meshes/link_r.STL" />
             </geometry>
-            <material name="">
-                <color rgba="1.0 1.0 1.0 1.0" />
-            </material>
         </visual>
         <collision>
@@ -92,6 +80,4 @@
         <child link="right_wheel" />
         <axis xyz="0 1 0" />
-        <limit effort="10000" velocity="1000"/>
-        <joint_properties damping="1.0" friction="1.0"/>
     </joint>
     <link name="camera">
@@ -109,7 +95,4 @@
                 <mesh filename="package://simulation/meshes/link_cam.STL" />
             </geometry>
-            <material name="">
-                <color rgba="1.0 1.0 1.0 1.0" />
-            </material>
         </visual>
         <collision>
