Commit message: Move robot on Gazebo

File: urdf/model.xacro (robot description, xacro)
@@ -1,4 +1,7 @@
-<?xml version="1.0" encoding="utf-8"?>
-<robot name="">
+<?xml version="1.0"?>
+<robot name="" xmlns:xacro="http://www.ros.org/wiki/xacro">
+    <!-- <xacro:property name="" value=""/> -->
+    <xacro:include filename="$(find simulation)/urdf/materials.xacro" />
+    <xacro:include filename="$(find simulation)/urdf/model.gazebo" />
     <link name="base_link">
         <inertial>

Commit message: Update README.md

File: urdf/model.xacro (robot description, xacro)
@@ -52,4 +52,6 @@
         <child link="left_wheel" />
         <axis xyz="0 1 0" />
+        <limit effort="1000" velocity="1000"/>
+        <joint_properties damping="1.0" friction="1.0"/>
     </joint>
     <link name="right_wheel">
@@ -80,4 +82,6 @@
         <child link="right_wheel" />
         <axis xyz="0 1 0" />
+        <limit effort="1000" velocity="1000"/>
+        <joint_properties damping="1.0" friction="1.0"/>
     </joint>
     <link name="camera">
